Commit message: Add files via upload
Set sim time in world file to zero and updates in pole

File: src/robotic_charger/urdf/pole2.xacro (robot description, xacro)
@@ -1,6 +1,6 @@
 <?xml version='1.0'?>
-<robot name="pole" xmlns:xacro="http://www.ros.org/wiki/xacro">
+<robot name="pole2" xmlns:xacro="http://www.ros.org/wiki/xacro">
   <!-- gazebo plugin files for sensors -->
-  <xacro:include filename="$(find robotic_charger)/urdf/pole.gazebo" />
+  <xacro:include filename="$(find robotic_charger)/urdf/pole2.gazebo" />
   <!-- Constants for robot dimensions -->
   <xacro:property name="PI" value="3.1415926535897931"/>
@@ -13,8 +13,8 @@
   <joint name="fixed" type="fixed">
     <parent link="world"/>
-    <child link="pole"/>
+    <child link="pole2"/>
   </joint>
   <!-- Base link -->
-  <link name='pole'>
+  <link name='pole2'>
     <pose>0 0 0 0 0 0</pose>
     <inertial>
@@ -33,5 +33,5 @@
       </geometry>
     </collision>
-    <visual name='pole_visual'>
+    <visual name='pole2_visual'>
       <origin xyz="0 0 ${height/2}" rpy=" 0 0 0"/>
       <geometry>
@@ -80,5 +80,5 @@
       <material>Gazebo/Green</material>
     </gazebo>
-    <gazebo reference="pole">
+    <gazebo reference="pole2">
       <material>Gazebo/Orange</material>
     </gazebo>

Commit message: Update pole2.xacro

File: src/robotic_charger/urdf/pole2.xacro (robot description, xacro)
@@ -42,5 +42,5 @@
       <axis xyz="0 1 0" />
       <origin xyz="${camera} 0 ${height}" rpy="0 0 0"/>
-      <parent link="link3"/>
+      <parent link="pole2"/>
       <child link="camera"/>
     </joint>
