Commit message: Update pole.xacro

File: src/robotic_charger/urdf/pole.xacro (robot description, xacro)
@@ -42,5 +42,5 @@
       <axis xyz="0 1 0" />
       <origin xyz="${camera} 0 ${height}" rpy="0 0 0"/>
-      <parent link="link3"/>
+      <parent link="pole"/>
       <child link="camera"/>
     </joint>

Commit message: Add files via upload

File: src/robotic_charger/urdf/pole.xacro (robot description, xacro)
@@ -7,6 +7,5 @@
   <xacro:property name="mass" value="100" /> <!-- arbitrary value for mass -->
   <xacro:property name="width" value="0.2" /> <!-- Square dimensions (widthxwidth) of beams -->
-  <xacro:property name="height" value="1.8" /> <!-- Link 1 -->
-  <xacro:property name="camera" value="0.1" /> <!-- Size of square 'camera' box -->
+  <xacro:property name="height" value="1.2" /> <!-- Link 1 -->
   <!-- Used for fixing pole to Gazebo 'base_link' -->
   <link name="world"/>
@@ -17,5 +16,4 @@
   <!-- Base link -->
   <link name='pole'>
-    <pose>0 0 0 0 0 0</pose>
     <inertial>
       <mass value="${mass}"/>
@@ -39,45 +37,4 @@
       </geometry>
     </visual>
-    <joint name="camera_joint" type="fixed">
-      <axis xyz="0 1 0" />
-      <origin xyz="${camera} 0 ${height}" rpy="0 0 0"/>
-      <parent link="pole"/>
-      <child link="camera"/>
-    </joint>
-    <!-- Camera -->
-    <link name="camera">
-      <collision>
-        <origin xyz="0 0 0" rpy="0 0 0"/>
-        <geometry>
-          <box size="${camera} ${camera} ${camera}"/>
-        </geometry>
-      </collision>
-      <visual>
-        <origin xyz="0 0 0" rpy="0 0 0"/>
-        <geometry>
-          <box size="${camera} ${camera} ${camera}"/>
-        </geometry>
-        <material name="green"/>
-      </visual>
-      <inertial>
-        <mass value="1e-5" />
-        <origin xyz="0 0 0" rpy="0 0 0"/>
-        <inertia ixx="1e-6" ixy="0" ixz="0" iyy="1e-6" iyz="0" izz="1e-6" />
-      </inertial>
-    </link>
-    <!-- generate an optical frame http://www.ros.org/reps/rep-0103.html#suffix-frames
-        so that ros and opencv can operate on the camera frame correctly -->
-    <joint name="camera_optical_joint" type="fixed">
-      <!-- these values have to be these values otherwise the gazebo camera image
-          won't be aligned properly with the frame it is supposedly originating from -->
-      <origin xyz="0 0 0" rpy="${-pi/2} 0 ${-pi/2}"/>
-      <parent link="camera"/>
-      <child link="camera_optical"/>
-    </joint>
-    <link name="camera_optical">
-    </link>
-    <gazebo reference="camera">
-      <material>Gazebo/Green</material>
-    </gazebo>
     <gazebo reference="pole">
       <material>Gazebo/Orange</material>

Commit message: Add files via upload

File: src/robotic_charger/urdf/pole.xacro (robot description, xacro)
@@ -8,4 +8,5 @@
   <xacro:property name="width" value="0.2" /> <!-- Square dimensions (widthxwidth) of beams -->
   <xacro:property name="height" value="1.2" /> <!-- Link 1 -->
+  <xacro:property name="camera" value="0.1" /> <!-- Size of square 'camera' box -->
   <!-- Used for fixing pole to Gazebo 'base_link' -->
   <link name="world"/>
@@ -37,7 +38,47 @@
       </geometry>
     </visual>
-    <gazebo reference="pole">
-      <material>Gazebo/Orange</material>
-    </gazebo>
   </link>
+  <joint name="camera_joint" type="fixed">
+      <axis xyz="0 1 0" />
+      <origin xyz="0 ${width/2} ${0.7*height} " rpy="0 0 0"/>
+      <parent link="pole"/>
+      <child link="pole_camera"/>
+  </joint>
+  <!-- Camera -->
+  <link name="pole_camera">
+    <collision>
+      <origin xyz="0 0 0" rpy="0 0 0"/>
+      <geometry>
+        <box size="${camera} ${camera} ${camera}"/>
+      </geometry>
+    </collision>
+    <visual>
+      <origin xyz="0 0 0" rpy="0 0 0"/>
+      <geometry>
+        <box size="${camera} ${camera} ${camera}"/>
+      </geometry>
+    </visual>
+    <inertial>
+      <mass value="1e-5" />
+      <origin xyz="0 0 0" rpy="0 0 0"/>
+      <inertia ixx="1e-6" ixy="0" ixz="0" iyy="1e-6" iyz="0" izz="1e-6" />
+    </inertial>
+  </link>
+  <!-- generate an optical frame http://www.ros.org/reps/rep-0103.html#suffix-frames
+      so that ros and opencv can operate on the camera frame correctly -->
+  <joint name="camera_optical_joint" type="fixed">
+    <!-- these values have to be these values otherwise the gazebo camera image
+        won't be aligned properly with the frame it is supposedly originating from -->
+    <origin xyz="0 0 0" rpy="${-pi/2} 0 ${-pi/2}"/>
+    <parent link="pole_camera"/>
+    <child link="camera_optical"/>
+  </joint>
+  <link name="camera_optical">
+  </link>
+  <gazebo reference="pole">
+    <material>Gazebo/Orange</material>
+  </gazebo>
+  <gazebo reference="pole_camera">
+    <material>Gazebo/Green</material>
+  </gazebo>
 </robot>

Commit message: Add files via upload

File: src/robotic_charger/urdf/pole.xacro (robot description, xacro)
@@ -7,5 +7,5 @@
   <xacro:property name="mass" value="100" /> <!-- arbitrary value for mass -->
   <xacro:property name="width" value="0.2" /> <!-- Square dimensions (widthxwidth) of beams -->
-  <xacro:property name="height" value="1.8" /> <!-- Link 1 -->
+  <xacro:property name="height" value="1.2" /> <!-- Link 1 -->
   <xacro:property name="camera" value="0.1" /> <!-- Size of square 'camera' box -->
   <!-- Used for fixing pole to Gazebo 'base_link' -->
@@ -17,5 +17,4 @@
   <!-- Base link -->
   <link name='pole'>
-    <pose>0 0 0 0 0 0</pose>
     <inertial>
       <mass value="${mass}"/>
@@ -39,48 +38,47 @@
       </geometry>
     </visual>
-    <joint name="camera_joint" type="fixed">
+  </link>
+  <joint name="camera_joint" type="fixed">
       <axis xyz="0 1 0" />
-      <origin xyz="${camera} 0 ${height}" rpy="0 0 0"/>
+      <origin xyz="0 ${width/2} ${0.7*height} " rpy="0 0 0"/>
       <parent link="pole"/>
-      <child link="camera"/>
-    </joint>
-    <!-- Camera -->
-    <link name="camera">
-      <collision>
-        <origin xyz="0 0 0" rpy="0 0 0"/>
-        <geometry>
-          <box size="${camera} ${camera} ${camera}"/>
-        </geometry>
-      </collision>
-      <visual>
-        <origin xyz="0 0 0" rpy="0 0 0"/>
-        <geometry>
-          <box size="${camera} ${camera} ${camera}"/>
-        </geometry>
-        <material name="green"/>
-      </visual>
-      <inertial>
-        <mass value="1e-5" />
-        <origin xyz="0 0 0" rpy="0 0 0"/>
-        <inertia ixx="1e-6" ixy="0" ixz="0" iyy="1e-6" iyz="0" izz="1e-6" />
-      </inertial>
-    </link>
-    <!-- generate an optical frame http://www.ros.org/reps/rep-0103.html#suffix-frames
-        so that ros and opencv can operate on the camera frame correctly -->
-    <joint name="camera_optical_joint" type="fixed">
-      <!-- these values have to be these values otherwise the gazebo camera image
-          won't be aligned properly with the frame it is supposedly originating from -->
-      <origin xyz="0 0 0" rpy="${-pi/2} 0 ${-pi/2}"/>
-      <parent link="camera"/>
-      <child link="camera_optical"/>
-    </joint>
-    <link name="camera_optical">
-    </link>
-    <gazebo reference="camera">
-      <material>Gazebo/Green</material>
-    </gazebo>
-    <gazebo reference="pole">
-      <material>Gazebo/Orange</material>
-    </gazebo>
+      <child link="pole_camera"/>
+  </joint>
+  <!-- Camera -->
+  <link name="pole_camera">
+    <collision>
+      <origin xyz="0 0 0" rpy="0 0 0"/>
+      <geometry>
+        <box size="${camera} ${camera} ${camera}"/>
+      </geometry>
+    </collision>
+    <visual>
+      <origin xyz="0 0 0" rpy="0 0 0"/>
+      <geometry>
+        <box size="${camera} ${camera} ${camera}"/>
+      </geometry>
+    </visual>
+    <inertial>
+      <mass value="1e-5" />
+      <origin xyz="0 0 0" rpy="0 0 0"/>
+      <inertia ixx="1e-6" ixy="0" ixz="0" iyy="1e-6" iyz="0" izz="1e-6" />
+    </inertial>
   </link>
+  <!-- generate an optical frame http://www.ros.org/reps/rep-0103.html#suffix-frames
+      so that ros and opencv can operate on the camera frame correctly -->
+  <joint name="camera_optical_joint" type="fixed">
+    <!-- these values have to be these values otherwise the gazebo camera image
+        won't be aligned properly with the frame it is supposedly originating from -->
+    <origin xyz="0 0 0" rpy="${-pi/2} 0 ${-pi/2}"/>
+    <parent link="pole_camera"/>
+    <child link="camera_optical"/>
+  </joint>
+  <link name="camera_optical">
+  </link>
+  <gazebo reference="pole">
+    <material>Gazebo/Orange</material>
+  </gazebo>
+  <gazebo reference="pole_camera">
+    <material>Gazebo/Green</material>
+  </gazebo>
 </robot>
