Commit message: fix base link of ur5 to ground

File: src/ur_description/urdf/inc/ur_macro.xacro (robot description, xacro)
@@ -316,4 +316,11 @@
       <child link="${prefix}tool0"/>
     </joint>
+    <!-- NEW addition -->
+    <!-- Used for fixing robot to Gazebo 'base_link' -->
+    <link name="world"/>
+    <joint name="fixed" type="fixed">
+      <parent link="world"/>
+      <child link="${prefix}base_link"/>
+    </joint>
   </xacro:macro>
 </robot>
